Commit message: Update arm configurations and fix joint types in URDF for Lula IK extension
- Modified left_arm.yaml and right_arm.yaml to update joint names.
- Adjusted scenario.py to correct the USD file path.
- Changed joint types from prismatic to fixed in xlerobot issac.urdf.
- Added new USD configuration files for the robot's components.

File: sim-issac/xlerobot_maniskill/xlerobot issac.urdf (robot description, URDF)
Before this commit: robot xlerobot, 32 links, 31 joints
Joints:
- joint root_x_axis_joint: type prismatic -> fixed
- joint root_y_axis_joint: type prismatic -> fixed
- joint root_z_rotation_joint: type continuous -> fixed
